Commit message: Add rosbag result

File: catkin_ws/src/dlv_description/urdf/dlv.urdf (robot description, URDF)
Before this commit: robot my_robot, 3 links, 2 joints
Joints:
- removed joint base_to_laser_joint
- joint base_to_base_footprint: child base_footprint -> base_link; parent base_link -> base_footprint
